File: examples/pcbs/mega_r3_sidecar_controller_rev_a.kicad_pcb (KiCad board)
At the start: 2 copper layers, 120.5 x 75 mm, 34 parts, among them J101 MCP2515 CTRL, J102 MAX31865, J103 CAN BUS, J104 ACT CMD, J105 COOL CALL, J106 LED HARNESS, J107 PWM RAW, J109 MCP2515 H/L, J111 24V IN, K1 AIR Z1, K2 AIR Z2, K3 AIR Z3, K4 AIR SPARE, K5 ACTUATOR, U201 5V REG MOD

Commit message: Normalize Arduino net aliases across wiring and preview UI
Connections:
- net /*44 renamed /PL4
- net /*45 renamed /PL5
- net /*46 renamed /PL2
- net /*52 renamed /PB0
- net /22 renamed /PA1
- net /23 renamed /PA0
- net /24 renamed /PA3
- net /25 renamed /PA2
- net /26 renamed /PA5
- net /27 renamed /PA4
- net /28 renamed /PA7
- net /29 renamed /PA6
- net /30 renamed /PC6
- net /31 renamed /PC7
- net /32 renamed /PC4
- net /33 renamed /PC5
- net /34 renamed /PC2
- net /35 renamed /PC3
- net /36 renamed /PC0
- net /37 renamed /PC1
- net /38 renamed /PG2
- net /39 renamed /PD7
- net /40 renamed /PG0
- net /41 renamed /PG1
- net /42 renamed /PL6
- net /43 renamed /PL7
- net /47 renamed /PL3
- net /48 renamed /PL0
- net /49 renamed /PL1
- net /50 renamed /PB2
- net /51 renamed /PB3
- net /53 renamed /PB1
- net /A10 renamed /ADC10
- net /A11 renamed /ADC11
- net /A12 renamed /ADC12
- net /A13 renamed /ADC13
- net /A14 renamed /ADC14
- net /A15 renamed /ADC15
- net /A8 renamed /ADC8
- net /A9 renamed /ADC9
